Commit message: feat: unlock gated csdog v2 locomotion training

File: source/stackforce_simready_generated_robot_lab/stackforce_simready_generated_robot_lab/assets/robots/csdog_v2/robot_sim.urdf (robot description, URDF)
Before this commit: robot robot, 17 links, 16 joints
Links:
- link link_lf_hip_pitch: geometry collision cylinder length=0.11569936 radius=0.022; collision sphere radius=0.048
- link link_lf_hip_roll: geometry collision cylinder length=0.025781333 radius=0.026; collision sphere radius=0.048
- link link_lf_knee: geometry collision cylinder length=0.089473416 radius=0.01; collision sphere radius=0.040
- link link_lr_hip_pitch: geometry collision cylinder length=0.11569936 radius=0.022; collision sphere radius=0.048
- link link_lr_hip_roll: geometry collision cylinder length=0.025781333 radius=0.026; collision sphere radius=0.048
- link link_lr_knee: geometry collision cylinder length=0.089468206 radius=0.01; collision sphere radius=0.040
- link link_rf_hip_pitch: geometry collision cylinder length=0.11569936 radius=0.022; collision sphere radius=0.048
- link link_rf_hip_roll: geometry collision cylinder length=0.025781333 radius=0.026; collision sphere radius=0.048
- link link_rf_knee: geometry collision cylinder length=0.089495344 radius=0.01; collision sphere radius=0.040
- link link_rr_hip_pitch: geometry collision cylinder length=0.11569937 radius=0.022; collision sphere radius=0.048
- link link_rr_hip_roll: geometry collision cylinder length=0.025781333 radius=0.026; collision sphere radius=0.048
- link link_rr_knee: geometry collision cylinder length=0.090318023 radius=0.01; collision sphere radius=0.040

Commit message: fix: make csdog sole contacts coplanar

File: source/stackforce_simready_generated_robot_lab/stackforce_simready_generated_robot_lab/assets/robots/csdog_v2/robot_sim.urdf (robot description, URDF)
Before this commit: robot robot, 17 links, 16 joints
Joints:
- joint joint_link_lf_sole_fixed: origin xyz=0.12389 0.00983 -0.16237 rpy=0 0 0 -> xyz=0.13702331 0.01025914 -0.16990075 rpy=0 0 0
- joint joint_link_lr_sole_fixed: origin xyz=0.11206 0.01206 -0.1706 rpy=0 0 0 -> xyz=0.10452175 0.01308119 -0.17931331 rpy=0 0 0
- joint joint_link_rf_sole_fixed: origin xyz=0.12364 -0.01044 -0.16255 rpy=0 0 0 -> xyz=0.11050669 -0.01001087 -0.16091365 rpy=0 0 0
- joint joint_link_rr_sole_fixed: origin xyz=0.08346 -0.01382 -0.18708 rpy=0 0 0 -> xyz=0.09099825 -0.01279881 -0.17247228 rpy=0 0 0
